Commit message: Added a goal entry for the dummy visualizer

File: ocs2_robotic_examples/ocs2_double_integrator_example/urdf/double_integrator.urdf (robot description, URDF)
Before this commit: robot double_integrator, 2 links, 1 joints
Links:
- added link goal, mass 1; collision box size=0.5 0.5 0.2; visual sphere radius=0.2
Joints:
- added joint slider_to_goal: type prismatic, parent slideBar, child goal, origin xyz=0.0 0.0 0.0, axis 1 0 0, limit lower=-150 upper=150 effort=100000.0 velocity=50

Commit message: doc is added.

File: ocs2_robotic_examples/ocs2_double_integrator_example/urdf/double_integrator.urdf (robot description, URDF)
Before this commit: robot double_integrator, 3 links, 2 joints
Links:
- removed link goal
- added link target, mass 1; collision box size=0.5 0.5 0.2; visual sphere radius=0.2
Joints:
- removed joint slider_to_goal
- added joint slider_to_target: type prismatic, parent slideBar, child target, origin xyz=0.0 0.0 0.0, axis 1 0 0, limit lower=-150 upper=150 effort=100000.0 velocity=50
