Commit message: raisim rollout working with cart-pole (hacky, hard-coded)

File: ocs2_robotic_examples/ocs2_cart_pole_example/urdf/cartpole.urdf (robot description, URDF)
Before this commit: robot cartpole, 3 links, 2 joints
Links:
- added link world
Joints:
- added joint world_to_slideBar: type fixed, parent world, child slideBar, origin xyz=0.0 0.0 0.0

Commit message: introduce new ocs2_raisim package, move cartpole raisim rollout into new package and add tests

File: ocs2_robotic_examples/ocs2_cart_pole_example/urdf/cartpole.urdf (robot description, URDF)
Before this commit: robot cartpole, 4 links, 3 joints
Joints:
- joint world_to_slideBar: origin xyz=0.0 0.0 0.0 -> xyz=0.0 0.0 2.0

Commit message: cartpole example is fixed

File: ocs2_robotic_examples/ocs2_cart_pole_example/urdf/cartpole.urdf (robot description, URDF)
Before this commit: robot cartpole, 4 links, 3 joints
Links:
- link cart: mass 1 -> 2.0
- link pole: mass 1 -> 0.2
