Commit message: Replaces the visuals with the collision geometry (which looks a bit more like the actual manipulator)

File: ocs2_robotic_examples/ocs2_mobile_manipulator_example/urdf/mobile_manipulator.urdf (robot description, URDF)
Before this commit: robot mm_arm, 9 links, 8 joints
Links:
- link ARM: geometry collision cylinder length=0.19 radius=0.07; collision cylinder length=0.22 radius=0.09
- link ELBOW: geometry collision cylinder length=0.46 radius=0.066; visual cylinder length=0.46 radius=0.066
- link FOREARM: geometry collision cylinder length=0.145 radius=0.05; collision cylinder length=0.25 radius=0.048
- link SHOULDER: geometry collision cylinder length=0.31 radius=0.09; visual cylinder length=0.31 radius=0.09
- link WRIST_1: geometry collision cylinder length=0.148 radius=0.05; visual cylinder length=0.148 radius=0.05
- link WRIST_2: geometry collision cylinder length=0.038 radius=0.05; visual cylinder length=0.038 radius=0.05

Commit message: Clean up gazebo stuff from URDF, rename world->base

File: ocs2_robotic_examples/ocs2_mobile_manipulator_example/urdf/mobile_manipulator.urdf (robot description, URDF)
Before this commit: robot mm_arm, 9 links, 8 joints
Links:
- removed link world
- added link base
Joints:
- joint world_to_arm_base: parent world -> base

Commit message: CppAD Quaternion conversion issue, update urdf, fix config, add base to pinocchio model

File: ocs2_robotic_examples/ocs2_mobile_manipulator_example/urdf/mobile_manipulator.urdf (robot description, URDF)
Before this commit: robot mm_arm, 9 links, 8 joints
Links:
- link arm_base: geometry collision box size=0.5 0.5 0.2; visual box size=0.5 0.5 0.2
Joints:
- joint world_to_arm_base: origin xyz=0 0 0.3 rpy=0 0 0 -> xyz=0 0 0.2 rpy=0 0 0

Commit message: Mostly debugging crap, also adds to the MobileManipulatorCost in a gross way

File: ocs2_robotic_examples/ocs2_mobile_manipulator_example/urdf/mobile_manipulator.urdf (robot description, URDF)
Before this commit: robot mm_arm, 9 links, 8 joints
Links:
- link arm_base: geometry collision box size=0.2 0.5 0.8; collision box size=0.5 0.5 0.2
