Commit message: update bear urdf

File: ocs2_anymal_models/kindsl/bear/cached_anymal_bear.urdf (robot description, URDF)
Before this commit: robot anymal, 33 links, 32 joints
Links:
- removed link realsense_d435_front_camera
- removed link realsense_d435_front_camera_axis_aligned
- removed link realsense_d435_front_camera_parent
- removed link realsense_d435_front_mount
- removed link realsense_d435_front_mount_tilted
- removed link velodyne
- removed link velodyne_axis_aligned
- removed link velodyne_mount
- added link depth_camera_front_camera, mass 0.072; collision box size=0.025 0.089 0.025; visual mesh filename=package://any_description/urdf/sensors/depth_camera/realsen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 scale=.001 .001 .001
- added link depth_camera_front_camera_axis_aligned
- added link depth_camera_front_camera_parent
- added link depth_camera_front_depth_optical_frame
- added link depth_camera_front_mount, mass 0.243898067
- added link depth_camera_front_mount_tilted, mass 0.015185133; collision box size=0.057 0.120 0.034; visual mesh filename=package://anymal_b/urdf/modules/depth_camera_mount/anymal_r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 scale=.001 .001 .001
- added link lidar, mass 0.01; visual mesh filename=package://velodyne_description/meshes/VLP16_scan.dae
- added link lidar_axis_aligned, mass 0.589004276; collision cylinder length=0.0717 radius=0.0516; visual mesh filename=package://velodyne_description/meshes/VLP16_base_1.dae
- added link lidar_mount, mass 0.468309149; collision cylinder length=0.15 radius=0.10; visual mesh filename=package://anymal_b/urdf/modules/lidar_mount/anymal_velodyne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 scale=.001 .001 .001
Joints:
- removed joint base_to_velodyne_mount
- removed joint handle_mount_front_sensor_mount_axis_aligned_to_realsense_d435_front_mount
- removed joint realsense_d435_front_camera_axis_aligned_to_camera
- removed joint realsense_d435_front_camera_to_camera_parent
- removed joint realsense_d435_front_mount_tilted_to_realsense_d435_front_camera_axis_aligned
- removed joint realsense_d435_front_mount_to_realsense_d435_front_mount_tilted
- removed joint velodyne_axis_aligned_to_velodyne
- removed joint velodyne_mount_to_velodyne_axis_aligned
- added joint base_to_lidar_mount: type fixed, parent base, child lidar_mount, origin xyz=-0.102 0.0 0.2896 rpy=0 0 0
- added joint depth_camera_front_camera_axis_aligned_to_camera: type fixed, parent depth_camera_front_camera_axis_aligned, child depth_camera_front_camera, origin xyz=0.0 0.0 0.0 rpy=0.0 0.0 0.0
- added joint depth_camera_front_camera_parent_to_depth_optical_frame: type fixed, parent depth_camera_front_camera_parent, child depth_camera_front_depth_optical_frame, origin xyz=0.0 0.0 0.0 rpy=-1.57079632679 0.0 -1.57079632679
- added joint depth_camera_front_camera_to_camera_parent: type fixed, parent depth_camera_front_camera, child depth_camera_front_camera_parent, origin xyz=0.02505 0.015 0.0125 rpy=0.0 0.0 0.0
- added joint depth_camera_front_mount_tilted_to_depth_camera_front_camera_axis_aligned: type fixed, parent depth_camera_front_mount_tilted, child depth_camera_front_camera_axis_aligned, origin xyz=0.013 0.0 -0.02362 rpy=0 0 0
- added joint depth_camera_front_mount_to_depth_camera_front_mount_tilted: type fixed, parent depth_camera_front_mount, child depth_camera_front_mount_tilted, origin xyz=0 0 0 rpy=0.0532019989239 0.614793974344 0.0
- added joint handle_mount_front_sensor_mount_axis_aligned_to_depth_camera_front_mount: type fixed, parent handle_mount_front_sensor_mount_axis_aligned, child depth_camera_front_mount, origin xyz=0.0 0.0 0.0 rpy=0.0 0.0 0.0
- added joint lidar_axis_aligned_to_velodyne: type fixed, parent lidar_axis_aligned, child lidar, origin xyz=0.0 0.0 0.0 rpy=0 0 0
- added joint lidar_mount_to_lidar_axis_aligned: type fixed, parent lidar_mount, child lidar_axis_aligned, origin xyz=0.0 0.0 0.0 rpy=0.0 0.0 -2.443460953
