Commit message: small fixes

File: ocs2_pinocchio/ocs2_centroidal_model/test/include/ocs2_centroidal_model/example/anymal/anymal.urdf (robot description, URDF)
Before this commit: robot anymal, 23 links, 22 joints
Links:
- removed link LF_ADAPTER
- removed link LH_ADAPTER
- removed link RF_ADAPTER
- removed link RH_ADAPTER
- added link LF_HAA, mass 2.04; visual mesh filename=package://anymal_c_simple_description/meshes/drive.dae scale=1.0 1.0 1.0
- added link LF_HFE, mass 2.04; collision cylinder length=0.14 radius=0.05; visual mesh filename=package://anymal_c_simple_description/meshes/drive.dae scale=1.0 1.0 1.0
- added link LF_KFE, mass 2.04; collision cylinder length=0.14 radius=0.05; visual mesh filename=package://anymal_c_simple_description/meshes/drive.dae scale=1.0 1.0 1.0
- added link LF_hip_fixed, mass 0.74; visual mesh filename=package://anymal_c_simple_description/meshes/hip_l.dae scale=1.0 1.0 1.0
- added link LF_shank_fixed, mass 0.33742; collision box size=0.114998 0.0675 0.04; collision cylinder length=0.04 radius=0.06
- added link LF_thigh_fixed, mass 1.03; collision box size=0.075 0.06 0.282627; collision cylinder length=0.08 radius=0.065
- added link LH_HAA, mass 2.04; visual mesh filename=package://anymal_c_simple_description/meshes/drive.dae scale=1.0 1.0 1.0
- added link LH_HFE, mass 2.04; collision cylinder length=0.14 radius=0.05; visual mesh filename=package://anymal_c_simple_description/meshes/drive.dae scale=1.0 1.0 1.0
- added link LH_KFE, mass 2.04; collision cylinder length=0.14 radius=0.05; visual mesh filename=package://anymal_c_simple_description/meshes/drive.dae scale=1.0 1.0 1.0
- added link LH_hip_fixed, mass 0.74; visual mesh filename=package://anymal_c_simple_description/meshes/hip_r.dae scale=1.0 1.0 1.0
- added link LH_shank_fixed, mass 0.33742; collision box size=0.114998 0.0675 0.04; collision cylinder length=0.04 radius=0.06
- added link LH_thigh_fixed, mass 1.03; collision box size=0.075 0.06 0.282627; collision cylinder length=0.08 radius=0.065
- added link RF_HAA, mass 2.04; visual mesh filename=package://anymal_c_simple_description/meshes/drive.dae scale=1.0 1.0 1.0
- added link RF_HFE, mass 2.04; collision cylinder length=0.14 radius=0.05; visual mesh filename=package://anymal_c_simple_description/meshes/drive.dae scale=1.0 1.0 1.0
- added link RF_KFE, mass 2.04; collision cylinder length=0.14 radius=0.05; visual mesh filename=package://anymal_c_simple_description/meshes/drive.dae scale=1.0 1.0 1.0
- added link RF_hip_fixed, mass 0.74; visual mesh filename=package://anymal_c_simple_description/meshes/hip_r.dae scale=1.0 1.0 1.0
- added link RF_shank_fixed, mass 0.33742; collision box size=0.114998 0.0675 0.04; collision cylinder length=0.04 radius=0.06
- added link RF_thigh_fixed, mass 1.03; collision box size=0.075 0.06 0.282627; collision cylinder length=0.08 radius=0.065
- added link RH_HAA, mass 2.04; visual mesh filename=package://anymal_c_simple_description/meshes/drive.dae scale=1.0 1.0 1.0
- added link RH_HFE, mass 2.04; collision cylinder length=0.14 radius=0.05; visual mesh filename=package://anymal_c_simple_description/meshes/drive.dae scale=1.0 1.0 1.0
- added link RH_KFE, mass 2.04; collision cylinder length=0.14 radius=0.05; visual mesh filename=package://anymal_c_simple_description/meshes/drive.dae scale=1.0 1.0 1.0
- added link RH_hip_fixed, mass 0.74; visual mesh filename=package://anymal_c_simple_description/meshes/hip_l.dae scale=1.0 1.0 1.0
- added link RH_shank_fixed, mass 0.33742; collision box size=0.114998 0.0675 0.04; collision cylinder length=0.04 radius=0.06
- added link RH_thigh_fixed, mass 1.03; collision box size=0.075 0.06 0.282627; collision cylinder length=0.08 radius=0.065
- added link battery, mass 5.53425; visual mesh filename=package://anymal_c_simple_description/meshes/battery.dae scale=1.0 1.0 1.0
- added link bottom_shell, mass 1.15; visual mesh filename=package://anymal_c_simple_description/meshes/bottom_shell.d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 scale=1.0 1.0 1.0
- added link depth_camera_front_camera, mass 0.16043; visual mesh filename=package://anymal_c_simple_description/meshes/depth_camera.d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 scale=1.0 1.0 1.0
- added link depth_camera_front_camera_parent
- added link depth_camera_front_color_frame
- added link depth_camera_front_color_optical_frame
- added link depth_camera_front_depth_optical_frame
- added link depth_camera_left_camera, mass 0.16043; visual mesh filename=package://anymal_c_simple_description/meshes/depth_camera.d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 scale=1.0 1.0 1.0
- added link depth_camera_left_camera_parent
- added link depth_camera_left_color_frame
- added link depth_camera_left_color_optical_frame
- added link depth_camera_left_depth_optical_frame
- added link depth_camera_rear_camera, mass 0.16043; visual mesh filename=package://anymal_c_simple_description/meshes/depth_camera.d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 scale=1.0 1.0 1.0
- added link depth_camera_rear_camera_parent
- added link depth_camera_rear_color_frame
- added link depth_camera_rear_color_optical_frame
- added link depth_camera_rear_depth_optical_frame
- added link depth_camera_right_camera, mass 0.16043; visual mesh filename=package://anymal_c_simple_description/meshes/depth_camera.d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 scale=1.0 1.0 1.0
- added link depth_camera_right_camera_parent
- added link depth_camera_right_color_frame
- added link depth_camera_right_color_optical_frame
- added link depth_camera_right_depth_optical_frame
- added link docking_hatch_cover, mass 0.065
- added link face_front, mass 0.73; collision box size=0.11 0.14 0.18; collision cylinder length=0.11 radius=0.09
- added link face_rear, mass 0.73; collision box size=0.11 0.14 0.18; collision cylinder length=0.11 radius=0.09
- added link handle, mass 0.314; visual mesh filename=package://anymal_c_simple_description/meshes/handle.dae scale=1.0 1.0 1.0
- added link hatch, mass 0.142; visual mesh filename=package://anymal_c_simple_description/meshes/hatch.dae scale=1.0 1.0 1.0
- added link lidar, mass 0.695; visual mesh filename=package://anymal_c_simple_description/meshes/lidar.dae
- added link lidar_cage, mass 0.545; collision cylinder length=0.12 radius=0.07; visual mesh filename=package://anymal_c_simple_description/meshes/lidar_cage.dae scale=1.0 1.0 1.0
- added link remote, mass 0.3262; visual mesh filename=package://anymal_c_simple_description/meshes/remote.dae scale=1.0 1.0 1.0
- added link top_shell, mass 0.534; visual mesh filename=package://anymal_c_simple_description/meshes/top_shell.dae scale=1.0 1.0 1.0
- added link wide_angle_camera_front_camera, mass 0.287; visual mesh filename=package://anymal_c_simple_description/meshes/wide_angle_cam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 scale=1.0 1.0 1.0
- added link wide_angle_camera_front_camera_parent
- added link wide_angle_camera_rear_camera, mass 0.287; visual mesh filename=package://anymal_c_simple_description/meshes/wide_angle_cam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 scale=1.0 1.0 1.0
- added link wide_angle_camera_rear_camera_parent
- link LF_FOOT: mass None -> 0.25; geometry collision cylinder length=0.282504 radius=0.0175; collision sphere radius=0.03
- link LF_HIP: mass 1.42462064 -> 0.001; geometry 
- link LF_SHANK: mass 0.207204302 -> 0.001; geometry 
- link LF_THIGH: mass 1.634976467 -> 0.001; geometry 
- link LH_FOOT: mass None -> 0.25; geometry collision cylinder length=0.282504 radius=0.0175; collision sphere radius=0.03
- link LH_HIP: mass 1.42462064 -> 0.001; geometry 
- link LH_SHANK: mass 0.207204302 -> 0.001; geometry 
- link LH_THIGH: mass 1.634976467 -> 0.001; geometry 
- link RF_FOOT: mass None -> 0.25; geometry collision cylinder length=0.282504 radius=0.0175; collision sphere radius=0.03
- link RF_HIP: mass 1.42462064 -> 0.001; geometry 
- link RF_SHANK: mass 0.207204302 -> 0.001; geometry 
- link RF_THIGH: mass 1.634976467 -> 0.001; geometry 
- link RH_FOOT: mass None -> 0.25; geometry collision cylinder length=0.282504 radius=0.0175; collision sphere radius=0.03
- link RH_HIP: mass 1.42462064 -> 0.001; geometry 
- link RH_SHANK: mass 0.207204302 -> 0.001; geometry 
- link RH_THIGH: mass 1.634976467 -> 0.001; geometry 
- link base: geometry collision box size=0.58 0.14 0.18; collision cylinder length=0.145 radius=0.09
- link base_inertia: mass 19.0 -> 6.222
- link imu_link: mass 0.05 -> 0.01; geometry collision box size=0.024 0.024 0.01; visual box size=0.024 0.024 0.01
Joints:
- removed joint LF_ADAPTER_TO_FOOT
- removed joint LF_SHANK_TO_ADAPTER
- removed joint LH_ADAPTER_TO_FOOT
- removed joint LH_SHANK_TO_ADAPTER
- removed joint RF_ADAPTER_TO_FOOT
- removed joint RF_SHANK_TO_ADAPTER
- removed joint RH_ADAPTER_TO_FOOT
- removed joint RH_SHANK_TO_ADAPTER
- added joint LF_HIP_LF_hip_fixed: type fixed, parent LF_HIP, child LF_hip_fixed, origin xyz=0 0 0 rpy=-2.61799387799 0 0.0
- added joint LF_THIGH_LF_thigh_fixed: type fixed, parent LF_THIGH, child LF_thigh_fixed, origin xyz=0 0 0 rpy=0 0 -1.57079632679
- added joint LF_hip_fixed_LF_HFE: type fixed, parent LF_hip_fixed, child LF_HFE, origin xyz=0.0599 0.08381 0.0 rpy=0 0 1.57079632679
- added joint LF_shank_LF_shank_fixed: type fixed, parent LF_SHANK, child LF_shank_fixed, origin xyz=0 0 0 rpy=0 0 -1.57079632679
- added joint LF_shank_fixed_LF_FOOT: type fixed, parent LF_shank_fixed, child LF_FOOT, origin xyz=0.08795 0.01305 -0.33797 rpy=0 0 0
- added joint LF_thigh_fixed_LF_KFE: type fixed, parent LF_thigh_fixed, child LF_KFE, origin xyz=0.0 0.1003 -0.285 rpy=0 0 1.57079632679
- added joint LH_HIP_LH_hip_fixed: type fixed, parent LH_HIP, child LH_hip_fixed, origin xyz=0 0 0 rpy=-2.61799387799 0 -3.14159265359
- added joint LH_THIGH_LH_thigh_fixed: type fixed, parent LH_THIGH, child LH_thigh_fixed, origin xyz=0 0 0 rpy=0 0 -1.57079632679
- added joint LH_hip_fixed_LH_HFE: type fixed, parent LH_hip_fixed, child LH_HFE, origin xyz=-0.0599 0.08381 0.0 rpy=0 0 1.57079632679
- added joint LH_shank_LH_shank_fixed: type fixed, parent LH_SHANK, child LH_shank_fixed, origin xyz=0 0 0 rpy=0 0 -1.57079632679
- added joint LH_shank_fixed_LH_FOOT: type fixed, parent LH_shank_fixed, child LH_FOOT, origin xyz=-0.08795 0.01305 -0.33797 rpy=0 0 0
- added joint LH_thigh_fixed_LH_KFE: type fixed, parent LH_thigh_fixed, child LH_KFE, origin xyz=-0.0 0.1003 -0.285 rpy=0 0 1.57079632679
- added joint RF_HIP_RF_hip_fixed: type fixed, parent RF_HIP, child RF_hip_fixed, origin xyz=0 0 0 rpy=2.61799387799 0 0.0
- added joint RF_THIGH_RF_thigh_fixed: type fixed, parent RF_THIGH, child RF_thigh_fixed, origin xyz=0 0 0 rpy=0 0 1.57079632679
- added joint RF_hip_fixed_RF_HFE: type fixed, parent RF_hip_fixed, child RF_HFE, origin xyz=0.0599 -0.08381 0.0 rpy=0 0 -1.57079632679
- added joint RF_shank_RF_shank_fixed: type fixed, parent RF_SHANK, child RF_shank_fixed, origin xyz=0 0 0 rpy=0 0 1.57079632679
- added joint RF_shank_fixed_RF_FOOT: type fixed, parent RF_shank_fixed, child RF_FOOT, origin xyz=0.08795 -0.01305 -0.33797 rpy=0 0 0
- added joint RF_thigh_fixed_RF_KFE: type fixed, parent RF_thigh_fixed, child RF_KFE, origin xyz=0.0 -0.1003 -0.285 rpy=0 0 -1.57079632679
- added joint RH_HIP_RH_hip_fixed: type fixed, parent RH_HIP, child RH_hip_fixed, origin xyz=0 0 0 rpy=2.61799387799 0 -3.14159265359
- added joint RH_THIGH_RH_thigh_fixed: type fixed, parent RH_THIGH, child RH_thigh_fixed, origin xyz=0 0 0 rpy=0 0 1.57079632679
- added joint RH_hip_fixed_RH_HFE: type fixed, parent RH_hip_fixed, child RH_HFE, origin xyz=-0.0599 -0.08381 0.0 rpy=0 0 -1.57079632679
- added joint RH_shank_RH_shank_fixed: type fixed, parent RH_SHANK, child RH_shank_fixed, origin xyz=0 0 0 rpy=0 0 1.57079632679
- added joint RH_shank_fixed_RH_FOOT: type fixed, parent RH_shank_fixed, child RH_FOOT, origin xyz=-0.08795 -0.01305 -0.33797 rpy=0 0 0
- added joint RH_thigh_fixed_RH_KFE: type fixed, parent RH_thigh_fixed, child RH_KFE, origin xyz=-0.0 -0.1003 -0.285 rpy=0 0 -1.57079632679
- added joint base_LF_HAA: type fixed, parent base, child LF_HAA, origin xyz=0.2999 0.104 0.0 rpy=2.61799387799 0 0.0
- added joint base_LH_HAA: type fixed, parent base, child LH_HAA, origin xyz=-0.2999 0.104 0.0 rpy=-2.61799387799 0 -3.14159265359
- added joint base_RF_HAA: type fixed, parent base, child RF_HAA, origin xyz=0.2999 -0.104 0.0 rpy=-2.61799387799 0 0.0
- added joint base_RH_HAA: type fixed, parent base, child RH_HAA, origin xyz=-0.2999 -0.104 0.0 rpy=2.61799387799 0 -3.14159265359
- added joint base_battery: type fixed, parent base, child battery, origin xyz=0 0 0 rpy=0 0 0
- added joint base_bottom_shell: type fixed, parent base, child bottom_shell, origin xyz=0 0 0 rpy=0 0 0
- added joint base_face_front: type fixed, parent base, child face_front, origin xyz=0.4145 0 0 rpy=0 0 -0.0
- added joint base_face_rear: type fixed, parent base, child face_rear, origin xyz=-0.4145 0 0 rpy=0 0 3.14159265359
- added joint base_handle: type fixed, parent base, child handle, origin xyz=0 0 0 rpy=0 0 0
- added joint base_hatch: type fixed, parent base, child hatch, origin xyz=0.0 0.0 0.0 rpy=0 0 0
- added joint base_remote: type fixed, parent base, child remote, origin xyz=0 0 0 rpy=0 0 0
- added joint base_to_depth_camera_left_camera: type fixed, parent base, child depth_camera_left_camera, origin xyz=0.0 0.07646 0.02905 rpy=0.0 0.523598775598 1.57079632679
- added joint base_to_depth_camera_right_camera: type fixed, parent base, child depth_camera_right_camera, origin xyz=0.0 -0.07646 0.02905 rpy=0.0 0.523598775598 -1.57079632679
- added joint base_to_docking_hatch_cover: type fixed, parent base, child docking_hatch_cover, origin xyz=0.343 0.0 -0.07 rpy=0 0 0
- added joint base_to_lidar_cage: type fixed, parent base, child lidar_cage, origin xyz=-0.364 0.0 0.0735 rpy=0 0 0
- added joint base_top_shell: type fixed, parent base, child top_shell, origin xyz=0 0 0 rpy=0 0 0
- added joint depth_camera_front_camera_parent_to_color_frame: type fixed, parent depth_camera_front_camera_parent, child depth_camera_front_color_frame, origin xyz=0 0.015 0 rpy=0 0 0
- added joint depth_camera_front_camera_parent_to_depth_optical_frame: type fixed, parent depth_camera_front_camera_parent, child depth_camera_front_depth_optical_frame, origin xyz=0.0 0.0 0.0 rpy=-1.57079632679 0.0 -1.57079632679
- added joint depth_camera_front_camera_to_camera_parent: type fixed, parent depth_camera_front_camera, child depth_camera_front_camera_parent, origin xyz=0.0255 0.0175 0.0 rpy=0.0 0.0 0.0
- added joint depth_camera_front_color_frame_to_color_optical_frame: type fixed, parent depth_camera_front_color_frame, child depth_camera_front_color_optical_frame, origin xyz=0.0 0.0 0.0 rpy=-1.57079632679 0.0 -1.57079632679
- added joint depth_camera_left_camera_parent_to_color_frame: type fixed, parent depth_camera_left_camera_parent, child depth_camera_left_color_frame, origin xyz=0 0.015 0 rpy=0 0 0
- added joint depth_camera_left_camera_parent_to_depth_optical_frame: type fixed, parent depth_camera_left_camera_parent, child depth_camera_left_depth_optical_frame, origin xyz=0.0 0.0 0.0 rpy=-1.57079632679 0.0 -1.57079632679
- added joint depth_camera_left_camera_to_camera_parent: type fixed, parent depth_camera_left_camera, child depth_camera_left_camera_parent, origin xyz=0.0255 0.0175 0.0 rpy=0.0 0.0 0.0
- added joint depth_camera_left_color_frame_to_color_optical_frame: type fixed, parent depth_camera_left_color_frame, child depth_camera_left_color_optical_frame, origin xyz=0.0 0.0 0.0 rpy=-1.57079632679 0.0 -1.57079632679
- added joint depth_camera_rear_camera_parent_to_color_frame: type fixed, parent depth_camera_rear_camera_parent, child depth_camera_rear_color_frame, origin xyz=0 0.015 0 rpy=0 0 0
- added joint depth_camera_rear_camera_parent_to_depth_optical_frame: type fixed, parent depth_camera_rear_camera_parent, child depth_camera_rear_depth_optical_frame, origin xyz=0.0 0.0 0.0 rpy=-1.57079632679 0.0 -1.57079632679
- added joint depth_camera_rear_camera_to_camera_parent: type fixed, parent depth_camera_rear_camera, child depth_camera_rear_camera_parent, origin xyz=0.0255 0.0175 0.0 rpy=0.0 0.0 0.0
- added joint depth_camera_rear_color_frame_to_color_optical_frame: type fixed, parent depth_camera_rear_color_frame, child depth_camera_rear_color_optical_frame, origin xyz=0.0 0.0 0.0 rpy=-1.57079632679 0.0 -1.57079632679
- added joint depth_camera_right_camera_parent_to_color_frame: type fixed, parent depth_camera_right_camera_parent, child depth_camera_right_color_frame, origin xyz=0 0.015 0 rpy=0 0 0
- added joint depth_camera_right_camera_parent_to_depth_optical_frame: type fixed, parent depth_camera_right_camera_parent, child depth_camera_right_depth_optical_frame, origin xyz=0.0 0.0 0.0 rpy=-1.57079632679 0.0 -1.57079632679
- added joint depth_camera_right_camera_to_camera_parent: type fixed, parent depth_camera_right_camera, child depth_camera_right_camera_parent, origin xyz=0.0255 0.0175 0.0 rpy=0.0 0.0 0.0
- added joint depth_camera_right_color_frame_to_color_optical_frame: type fixed, parent depth_camera_right_color_frame, child depth_camera_right_color_optical_frame, origin xyz=0.0 0.0 0.0 rpy=-1.57079632679 0.0 -1.57079632679
- added joint face_front_to_depth_camera_front_camera: type fixed, parent face_front, child depth_camera_front_camera, origin xyz=0.04715 0.0 -0.0292 rpy=0.0 0.523598775598 0
- added joint face_front_to_wide_angle_camera_front_camera: type fixed, parent face_front, child wide_angle_camera_front_camera, origin xyz=0.09850 0.0 0.01497 rpy=0 0 0
- added joint face_rear_to_depth_camera_rear_camera: type fixed, parent face_rear, child depth_camera_rear_camera, origin xyz=0.04715 0.0 -0.0292 rpy=0.0 0.523598775598 0
- added joint face_rear_to_wide_angle_camera_rear_camera: type fixed, parent face_rear, child wide_angle_camera_rear_camera, origin xyz=0.09850 0.0 0.01497 rpy=0 0 0
- added joint lidar_cage_to_lidar: type fixed, parent lidar_cage, child lidar, origin xyz=0.0 0.0 0.0687 rpy=0.0 0.0 -1.57079632679
- added joint wide_angle_camera_front_camera_to_camera_parent: type fixed, parent wide_angle_camera_front_camera, child wide_angle_camera_front_camera_parent, origin xyz=0.0 0.0 0.0 rpy=-1.57079632679 0.0 -1.57079632679
- added joint wide_angle_camera_rear_camera_to_camera_parent: type fixed, parent wide_angle_camera_rear_camera, child wide_angle_camera_rear_camera_parent, origin xyz=0.0 0.0 0.0 rpy=-1.57079632679 0.0 -1.57079632679
- joint LF_HAA: limit lower=-9.42 upper=9.42 effort=80 velocity=15 -> lower=-0.72 upper=0.49 effort=80.0 velocity=7.5; origin xyz=0.277 0.116 0.0 -> xyz=0 0 0 rpy=0 0 0; parent base -> LF_HAA
- joint LF_HFE: axis 0 1 0 -> 1 0 0; limit lower=-9.42 upper=9.42 effort=80 velocity=15.0 -> lower=-9.42477796077 upper=9.42477796077 effort=80.0 velocity=7.5; origin xyz=0.0635                    0.041                    0.0 -> xyz=0 0 0 rpy=0 0 0; parent LF_HIP -> LF_HFE
- joint LF_KFE: axis 0 1 0 -> 1 0 0; limit lower=-9.42 upper=9.42 effort=80 velocity=15.0 -> lower=-9.42477796077 upper=9.42477796077 effort=80.0 velocity=7.5; origin xyz=0.0 0.109 -0.25 -> xyz=0 0 0 rpy=0 0 0; parent LF_THIGH -> LF_KFE
- joint LH_HAA: axis 1 0 0 -> -1 0 0; limit lower=-9.42 upper=9.42 effort=80 velocity=15 -> lower=-0.72 upper=0.49 effort=80.0 velocity=7.5; origin xyz=-0.277 0.116 0.0 -> xyz=0 0 0 rpy=0 0 0; parent base -> LH_HAA
- joint LH_HFE: axis 0 1 0 -> 1 0 0; limit lower=-9.42 upper=9.42 effort=80 velocity=15.0 -> lower=-9.42477796077 upper=9.42477796077 effort=80.0 velocity=7.5; origin xyz=-0.0635                    0.041                    0.0 -> xyz=0 0 0 rpy=0 0 0; parent LH_HIP -> LH_HFE
- joint LH_KFE: axis 0 1 0 -> 1 0 0; limit lower=-9.42 upper=9.42 effort=80 velocity=15.0 -> lower=-9.42477796077 upper=9.42477796077 effort=80.0 velocity=7.5; origin xyz=-0.0 0.109 -0.25 -> xyz=0 0 0 rpy=0 0 0; parent LH_THIGH -> LH_KFE
- joint RF_HAA: limit lower=-9.42 upper=9.42 effort=80 velocity=15 -> lower=-0.49 upper=0.72 effort=80.0 velocity=7.5; origin xyz=0.277 -0.116 0.0 -> xyz=0 0 0 rpy=0 0 0; parent base -> RF_HAA
- joint RF_HFE: axis 0 1 0 -> -1 0 0; limit lower=-9.42 upper=9.42 effort=80 velocity=15.0 -> lower=-9.42477796077 upper=9.42477796077 effort=80.0 velocity=7.5; origin xyz=0.0635                    -0.041                    0.0 -> xyz=0 0 0 rpy=0 0 0; parent RF_HIP -> RF_HFE
- joint RF_KFE: axis 0 1 0 -> -1 0 0; limit lower=-9.42 upper=9.42 effort=80 velocity=15.0 -> lower=-9.42477796077 upper=9.42477796077 effort=80.0 velocity=7.5; origin xyz=0.0 -0.109 -0.25 -> xyz=0 0 0 rpy=0 0 0; parent RF_THIGH -> RF_KFE
- joint RH_HAA: axis 1 0 0 -> -1 0 0; limit lower=-9.42 upper=9.42 effort=80 velocity=15 -> lower=-0.49 upper=0.72 effort=80.0 velocity=7.5; origin xyz=-0.277 -0.116 0.0 -> xyz=0 0 0 rpy=0 0 0; parent base -> RH_HAA
- joint RH_HFE: axis 0 1 0 -> -1 0 0; limit lower=-9.42 upper=9.42 effort=80 velocity=15.0 -> lower=-9.42477796077 upper=9.42477796077 effort=80.0 velocity=7.5; origin xyz=-0.0635                    -0.041                    0.0 -> xyz=0 0 0 rpy=0 0 0; parent RH_HIP -> RH_HFE
- joint RH_KFE: axis 0 1 0 -> -1 0 0; limit lower=-9.42 upper=9.42 effort=80 velocity=15.0 -> lower=-9.42477796077 upper=9.42477796077 effort=80.0 velocity=7.5; origin xyz=-0.0 -0.109 -0.25 -> xyz=0 0 0 rpy=0 0 0; parent RH_THIGH -> RH_KFE
- joint imu_joint: origin xyz=0.062 0.05755 0.1837 rpy=3.14159265359 0 0 -> xyz=0.2488 0.00835 0.04628 rpy=0.0 0.0 1.57079632679
