Commit message: adding ocs2_robotic_assets and moving urdf to this package

File: ocs2_robotic_assets/resources/ballbot/urdf/ballbot.urdf (robot description, URDF)
Before this commit: robot ballbot, 7 links, 6 joints
Links:
- link base: geometry visual mesh filename=package://ocs2_robotic_assets/resources/ballbot/meshes/base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 scale=1.0 1.0 1.0

File: ocs2_robotic_assets/resources/quadrotor/urdf/quadrotor.urdf (robot description, URDF)
Before this commit: robot quadrotor, 1 links, 0 joints
Links:
- link base: geometry collision cylinder length=.1 radius=.3; visual mesh filename=file://$(find ocs2_robotic_assets)/resources/quadrotor/mesh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 scale=.4 .4 .4
