Commit message: Adding an extra collision body for the base of the dummy urdf

File: ocs2_pinocchio/ocs2_sphere_approximation/urdf/dummy.urdf (robot description, URDF)
Before this commit: robot dummy, 5 links, 4 joints
Links:
- link base: geometry collision box size=0.2 0.2 0.2; collision box size=1.0 0.5 0.3
