Commit message: remove chimera and cerberus

File: ocs2_robotic_examples/ocs2_perceptive_anymal/ocs2_anymal_models/urdf/anymal_camel_rsl.urdf (robot description, URDF)
Before this commit: robot anymal, 69 links, 68 joints
Links:
- link interface_hatch: geometry collision box size=0.1817832 0.1296570 0.055
- link perception_head_cage: geometry collision box size=0.14151 0.21544 0.1768
